File: BLDC_MOTOR_DRIVER_V0.kicad_sch (KiCad schematic)
At the start: 54 parts, among them J1 Conn_01x05_Pin, J10 Conn_01x01_Socket, J11 Conn_01x01_Socket, J12 Conn_01x01_Socket, J13 Conn_01x01_Socket, J14 Conn_01x01_Socket, J2 Conn_01x01_Socket, J3 Conn_01x01_Socket, J4 Conn_01x01_Socket, J5 Conn_01x01_Socket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

Commit message: dg
Parts:
- removed Q1, Q2, Q3, Q4, Q5, Q6: N-MOSFET, NTMFS5C468NLT1G:NTMFS5C468NLT1G, symbol NTMFS5C468NLT1G:NTMFS5C468NLT1G
- added Q1, Q2, Q3: N-MOS Half-Bridge, CSD87588N:CSD87588N, symbol CSD87588N:CSD87588N
Connections:
- net +BATT: now also Q1.2 (Vin), Q2.2 (Vin), Q3.2 (Vin)
- net GHA: now also Q1.1 (TG)
- net GHB: now also Q2.1 (TG)
- net GHC: now also Q3.1 (TG)
- net GLA: now also Q1.4 (BG)
- net GLB: now also Q2.4 (BG)
- net GLC: now also Q3.4 (BG)
- net MOTOR_A: now also Q1.5 (SW)
- net MOTOR_B: now also Q2.5 (SW)
- net MOTOR_C: now also Q3.5 (SW)
- net SPA: now also Q1.3 (Vout)
- net SPB: now also Q2.3 (Vout)
- net SPC: now also Q3.3 (Vout)
Other:
- moved on the sheet: C10, C11, C12, C17, C21, C22, R3, R4, R5

Commit message: ap
Connections:
- net HA: now also U2.2 (AD1AN6/RP8/IOMF1/RA7); no longer U2.8 (OA1OUT/AD1AN0/CMP1A/RP3/RA2)
- net HB: now also U2.5 (AD1ANN3/AD1AN9/RP10/RA9); no longer U2.10 (OA1IN+/AD1AN1/CMP1B/RP5/RA4)
- net HC: now also U2.8 (OA1OUT/AD1AN0/CMP1A/RP3/RA2); no longer U2.12 (OA3IN-/AD1AN2/RP7/RA6)

Commit message: af
Parts:
- added J15, J16: Conn_01x01_Socket, Connector_Wire:SolderWirePad_1x01_SMD_2x4mm, symbol Connector:Conn_01x01_Socket
Connections:
- net -BATT: now also J15.1 (Pin_1)
- net VDC: now also J16.1 (Pin_1)
Other:
- moved on the sheet: J10, J8, J9

Commit message: update
Connections:
- net HA: now also U2.16 (OA2OUT/AD2AN1/CMP2A/RP17/INT0/RB0); no longer U2.2 (AD1AN6/RP8/IOMF1/RA7)
- net HB: now also U2.18 (OA2IN+/AD2AN4/CMP2B/RP19/RB2); no longer U2.5 (AD1ANN3/AD1AN9/RP10/RA9)
- net HC: now also U2.22 (PGC1/AD2AN5/CMP2C/ISRC1/IBIAS1/RP21/SCL1/RB4); no longer U2.8 (OA1OUT/AD1AN0/CMP1A/RP3/RA2)
- net LVDS_DE: now also U2.28 (OSCI/CLKI/RP34/IOMF6/RC1); no longer U2.25 (RP39/RC6)
- net LVDS_DI: now also U2.27 (OSCO/CLKO/RP33/IOMF5/RC0); no longer U2.26 (RP40/RC7)
- net LVDS_RE: now also U2.25 (RP39/RC6); no longer U2.27 (OSCO/CLKO/RP33/IOMF5/RC0)
- net LVDS_RO: now also U2.26 (RP40/RC7); no longer U2.28 (OSCI/CLKI/RP34/IOMF6/RC1)
- net SOA: now also U2.2 (AD1AN6/RP8/IOMF1/RA7); no longer U2.16 (OA2OUT/AD2AN1/CMP2A/RP17/INT0/RB0)
- net SOB: now also U2.5 (AD1ANN3/AD1AN9/RP10/RA9); no longer U2.18 (OA2IN+/AD2AN4/CMP2B/RP19/RB2)
- net SOC: now also U2.8 (OA1OUT/AD1AN0/CMP1A/RP3/RA2); no longer U2.22 (PGC1/AD2AN5/CMP2C/ISRC1/IBIAS1/RP21/SCL1/RB4)

Commit message: fgn
Parts:
- removed C16, C20: 10uF, Capacitor_SMD:C_Elec_5x5.4, symbol EMK1VM100D80D00R:EMK1VM100D80D00R
- added C16, C19: 22uF, Capacitor_SMD:CP_Elec_5x5.3, symbol 865080542006:865080542006
Connections:
- net +BATT: now also C16.1, C19.1
- net -BATT: now also C16.2, C19.2
Changed lines of the file:
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@@
 	)
 	(junction
+		(at 120.65 267.97)
+		(diameter 0)
+		(color 0 0 0 0)
+	)
+	(junction
 		(at 236.22 68.58)
 		(diameter 0)
@@
 	)
 	(junction
-		(at 121.92 267.97)
+		(at 120.65 260.35)
 		(diameter 0)
 		(color 0 0 0 0)
@@
 	)
 	(junction
-		(at 121.92 260.35)
-		(diameter 0)
-		(color 0 0 0 0)
-	)
-	(junction
 		(at 59.69 205.74)
 		(diameter 0)
@@
 	(wire
 		(pts
-			(xy 121.92 267.97) (xy 138.43 267.97)
+			(xy 118.11 267.97) (xy 120.65 267.97)
 		)
 		(stroke
@@
 	(wire
 		(pts
-			(xy 133.35 260.35) (xy 121.92 260.35)
-		)
-		(stroke
-			(width 0)
-			(type default)
-		)
-	)
-	(wire
-		(pts
 			(xy 327.66 104.14) (xy 327.66 105.41)
 		)
@@
 	(wire
 		(pts
-			(xy 118.11 260.35) (xy 121.92 260.35)
+			(xy 118.11 260.35) (xy 120.65 260.35)
 		)
 		(stroke
@@
 	(wire
 		(pts
+			(xy 120.65 267.97) (xy 138.43 267.97)
+		)
+		(stroke
+			(width 0)
+			(type default)
+		)
+	)
+	(wire
+		(pts
 			(xy 222.25 81.28) (xy 220.98 81.28)
 		)
@@
 	(wire
 		(pts
-			(xy 377.19 185.42) (xy 364.49 185.42)
+			(xy 120.65 260.35) (xy 133.35 260.35)
 		)
 		(stroke
@@
 	(wire
 		(pts
-			(xy 337.82 96.52) (xy 337.82 95.25)
+			(xy 377.19 185.42) (xy 364.49 185.42)
 		)
 		(stroke
@@
 	(wire
 		(pts
-			(xy 59.69 196.85) (xy 48.26 196.85)
+			(xy 337.82 96.52) (xy 337.82 95.25)
 		)
 		(stroke
@@
 	(wire
 		(pts
-			(xy 118.11 267.97) (xy 121.92 267.97)
+			(xy 59.69 196.85) (xy 48.26 196.85)
 		)
 		(stroke
@@
 	)
 	(symbol
+		(lib_id "865080542006:865080542006")
+		(at 120.65 264.16 0)
+		(unit 1)
+		(exclude_from_sim no)
+		(in_bom yes)
+		(on_board yes)
+		(dnp no)
+		(fields_autoplaced yes)
+		(property "Reference" "C19"
+			(at 124.46 262.0009 0)
+			(effects
+				(font
+					(size 1.27 1.27)
+				)
+				(justify left)
+			)
+		)
+		(property "Value" "22uF"
+			(at 124.46 264.5409 0)
+			(effects
+				(font
+					(size 1.27 1.27)
+				)
+				(justify left)
+			)
+		)
+		(property "Footprint" "Capacitor_SMD:CP_Elec_5x5.3"
+			(at 119.126 268.478 0)
+			(effects
+				(font
+					(size 1.27 1.27)
+				)
+				(hide yes)
+			)
+		)
+		(property "Datasheet" "https://www.we-online.com/components/products/datasheet/865080542006.pdf"
+			(at 119.126 268.478 0)
+			(effects
+				(font
+					(size 1.27 1.27)
+				)
+				(hide yes)
+			)
+		)
+		(property "Description" "22uF 35V"
+			(at 120.65 264.16 0)
+			(effects
+				(font
+					(size 1.27 1.27)
+				)
+				(hide yes)
+			)
+		)
+		(property "product" "865080542006"
+			(at 119.126 268.478 0)
+			(effects
+				(font
+					(size 1.27 1.27)
+				)
+				(hide yes)
+			)
+		)
+		(pin "2"
+		)
+		(pin "1"
+		)
+		(instances
+			(project "BLDC_MOTOR_DRIVER_V0"
+				(path "/f8ba6892-ec81-43be-a77b-cb45d1b0b522"
+					(reference "C19")
+					(unit 1)
+				)
+			)
+		)
+	)
+	(symbol
 		(lib_id "power:GND")
 		(at 128.27 224.79 0)
@@
 	)
 	(symbol
-		(lib_id "EMK1VM100D80D00R:EMK1VM100D80D00R")
-		(at 274.32 148.59 0)
-		(unit 1)
-		(exclude_from_sim no)
-		(in_bom yes)
-		(on_board yes)
-		(dnp no)
-		(property "Reference" "C16"
-			(at 279.4 147.32 0)
-			(effects
-				(font
-					(size 1.27 1.27)
-				)
-			)
-		)
-		(property "Value" "10uF"
-			(at 279.4 149.86 0)
-			(effects
-				(font
-					(size 1.27 1.27)
-				)
-			)
-		)
-		(property "Footprint" "Capacitor_SMD:C_Elec_5x5.4"
-			(at 274.32 148.59 0)
-			(effects
-				(font
-					(size 1.27 1.27)
-				)
-				(hide yes)
-			)
-		)
-		(property "Datasheet" "https://mm.digikey.com/Volume0/opasdata/d220001/medias/docus/7696/MK.pdf"
-			(at 274.32 148.59 0)
-			(effects
-				(font
-					(size 1.27 1.27)
-				)
-				(hide yes)
-			)
-		)
-		(property "Description" "capaciter 10uF 35V"
-			(at 274.32 148.59 0)
-			(effects
-				(font
-					(size 1.27 1.27)
-				)
-				(hide yes)
-			)
-		)
-		(property "product" "EMK1VM100D80D00R"
-			(at 274.32 148.59 0)
-			(effects
-				(font
-					(size 1.27 1.27)
-				)
-				(hide yes)
-			)
-		)
-		(pin "1"
-		)
-		(pin "2"
-		)
-		(instances
-			(project "BLDC_MOTOR_DRIVER_V0"
-				(path "/f8ba6892-ec81-43be-a77b-cb45d1b0b522"
-					(reference "C16")
-					(unit 1)
-				)
-			)
-		)
-	)
-	(symbol
 		(lib_id "CGA2B3X7R1H473K050BB:CGA2B3X7R1H473K050BB")
 		(at 306.07 130.81 0)
@@
 	)
 	(symbol
-		(lib_id "EMK1VM100D80D00R:EMK1VM100D80D00R")
-		(at 121.92 264.16 0)
-		(unit 1)
-		(exclude_from_sim no)
-		(in_bom yes)
-		(on_board yes)
-		(dnp no)
-		(fields_autoplaced yes)
-		(property "Reference" "C20"
-			(at 125.73 262.0009 0)
-			(effects
-				(font
-					(size 1.27 1.27)
-				)
-				(justify left)
-			)
-		)
-		(property "Value" "10uF"
-			(at 125.73 264.5409 0)
-			(effects
-				(font
-					(size 1.27 1.27)
-				)
-				(justify left)
-			)
-		)
-		(property "Footprint" "Capacitor_SMD:C_Elec_5x5.4"
-			(at 121.92 264.16 0)
-			(effects
-				(font
-					(size 1.27 1.27)
-				)
-				(hide yes)
-			)
-		)
-		(property "Datasheet" "https://mm.digikey.com/Volume0/opasdata/d220001/medias/docus/7696/MK.pdf"
-			(at 121.92 264.16 0)
-			(effects
-				(font
-					(size 1.27 1.27)
-				)
-				(hide yes)
-			)
-		)
-		(property "Description" "capaciter 10uF 35V"
-			(at 121.92 264.16 0)
-			(effects
-				(font
-					(size 1.27 1.27)
-				)
-				(hide yes)
-			)
-		)
-		(property "product" "EMK1VM100D80D00R"
-			(at 121.92 264.16 0)
-			(effects
-				(font
-					(size 1.27 1.27)
-				)
-				(hide yes)
-			)
-		)
-		(pin "1"
-		)
-		(pin "2"
-		)
-		(instances
-			(project "BLDC_MOTOR_DRIVER_V0"
-				(path "/f8ba6892-ec81-43be-a77b-cb45d1b0b522"
-					(reference "C20")
-					(unit 1)
-				)
-			)
-		)
-	)
-	(symbol
 		(lib_id "CSD87588N:CSD87588N")
 		(at 339.09 85.09 0)
@@
 					(unit 1)
 				)
+			)
+		)
+	)
+	(symbol
+		(lib_id "865080542006:865080542006")
+		(at 274.32 148.59 0)
+		(unit 1)
+		(exclude_from_sim no)
+		(in_bom yes)
+		(on_board yes)
+		(dnp no)
+		(fields_autoplaced yes)
+		(property "Reference" "C16"
+			(at 278.13 146.4309 0)
+			(effects
+				(font
+					(size 1.27 1.27)
+				)
+				(justify left)
+			)
+		)
+		(property "Value" "22uF"
+			(at 278.13 148.9709 0)
+			(effects
+				(font
+					(size 1.27 1.27)
+				)
+				(justify left)
+			)
+		)
+		(property "Footprint" "Capacitor_SMD:CP_Elec_5x5.3"
+			(at 272.796 152.908 0)
+			(effects
+				(font
+					(size 1.27 1.27)
+				)
+				(hide yes)
+			)
+		)
+		(property "Datasheet" "https://www.we-online.com/components/products/datasheet/865080542006.pdf"
+			(at 272.796 152.908 0)
+			(effects
+				(font
+					(size 1.27 1.27)
+				)
+				(hide yes)
+			)
+		)
+		(property "Description" "22uF 35V"
+			(at 274.32 148.59 0)
+			(effects
+				(font
+					(size 1.27 1.27)
+				)
+				(hide yes)
+			)
+		)
+		(property "product" "865080542006"
+			(at 272.796 152.908 0)
+			(effects
+				(font
+					(size 1.27 1.27)
+				)
+				(hide yes)
+			)
+		)
+		(pin "2"
+		)
+		(pin "1"
+		)
+		(instances
+			(project ""
+				(path "/f8ba6892-ec81-43be-a77b-cb45d1b0b522"
+					(reference "C16")
+					(unit 1)
+				)

Commit message: up
Parts:
- added R8: 10k, Resistor_SMD:R_0603_1608Metric, symbol NRC06F1002TRF:NRC06F1002TRF
- C1, C13, C14, C15, C17, C18, C2, C21, C22, C3, C4, C5, C6: digikey (none) -> none
- C10, C11, C12: digikey (none) -> 311-1083-1-ND
- C16, C19: digikey (none) -> 732-8505-1-ND
- C23, C24, C8, C9: digikey (none) -> 1276-1029-1-ND
- C7: digikey (none) -> 445-6897-1-ND
- J1, J10, J11, J12, J13, J14, J15, J16, J2, J3, J4, J5, J6, J7, J8, J9: now left out of the parts list
- Q1, Q2, Q3: digikey (none) -> 296-35792-1-ND
- R1, R2, R6, R7: digikey (none) -> 4988-NRC06F1002TRFCT-ND
- R3, R4, R5: digikey (none) -> 738-CSNL2512FTL300CT-ND
- U1: digikey (none) -> 264-TB67Z833SFTG(O,EL)CT-ND
- U2: symbol DSPIC33AK32MC105:DSPIC33AK32MC105 -> DSPIC33AK32MC105-IPT:DSPIC33AK32MC105-I/PT; digikey (none) -> 150-DSPIC33AK32MC105-I/PT-ND; product DSPIC33AK32MC105 -> DSPIC33AK32MC105-I/PT
- U4: digikey (none) -> 296-TLV74033PDBVRCT-ND
- U5: digikey (none) -> FIN1019MTCXCT-ND
Connections:
- net -BATT: now also R8.1
- net MCU_NC: now reaches U2.10 (OA1IN+/AD1AN1/CMP1B/RP5/RA4)
- net MCU_NC: now also U2.11 (OA3OUT/AD1AN3/CMP3A/RP6/RA5), U2.12 (OA3IN-/AD1AN2/RP7/RA6), U2.13 (OA3IN+/AD2AN2/CMP3B/RP22/RB5), U2.17 (TMS/OA2IN-/AD1AN4/AD2ANN1/RP18/RB1), U2.21 (PGD1/AD1AN5/CMP1C/ISRC0/IBIAS0/RP20/SDA1/RB3), U2.23 (AD1ANN2/AD1AN8/RP23/RB6), U2.24 (AD2ANN2/AD2AN8/RP24/IOMF0/RB7), U2.4 (AD2AN9/ISRC3/IBIAS3/RP9/RA8), U2.47 (RP53/PCI22/RD4), U2.9 (OA1IN-/AD1ANN1/AD2AN0/RP4/RA3), R8.2
Other:
- moved on the sheet: C1

Commit message: v1.0.0
Parts:
- added R9: 100, Resistor_SMD:R_0402_1005Metric, symbol RK73H1ETTP1000F:RK73H1ETTP1000F
Connections:
- net LVDS_RI+: now also R9.1
- net LVDS_RI-: now also R9.2
Other:
- note added: "3phase invertar"
- note added: "CONNECTOR"
- note added: "GateDriver"
- note added: "HOLE"
- note added: "LVDS"
- note added: "MCU"
- note added: "MOTER"
- note added: "NC"
- note added: "PICKIT"
- note added: "POWER"
- note added: "REGURATOR"
- moved on the sheet: C1, C13, C14, C15, C16, C18, C19, C2, C23, C24, C3, C4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
