File: BLDC_MOTOR_DRIVER_V0.kicad_pcb (KiCad board)
At the start: 2 copper layers, 30 x 60 mm, 34 parts, among them Q1 N-MOSFET, Q2 N-MOSFET, Q3 N-MOSFET, Q4 N-MOSFET, Q5 N-MOSFET, Q6 N-MOSFET, U1 3-phase Gate Driver, U2 Micro controller

Commit message: update
Parts:
- removed C100: 10uF, Capacitor_SMD:C_Elec_5x5.4
- removed R100: 1k, Resistor_SMD:R_0603_1608Metric
- removed REF** (x4): MountingHole_3.2mm_M3_DIN965, MountingHole:MountingHole_3.2mm_M3_DIN965
- added C16: 10uF, Capacitor_SMD:C_Elec_5x5.4, F.Cu at (192.8, 73.5)
- added C17: 0.1uF, Capacitor_SMD:C_0603_1608Metric, F.Cu at (171.9, 90.7)
- added C18: 10uF, Capacitor_SMD:C_Elec_5x5.4, F.Cu at (185.0, 33.0)
- added C19: 10uF, Capacitor_SMD:C_Elec_5x5.4, F.Cu at (185.5, 44.5)
- added C20: 10uF, Capacitor_SMD:C_Elec_5x5.4, F.Cu at (175.5, 34.0)
- added C21: 0.1uF, Capacitor_SMD:C_0603_1608Metric, F.Cu at (182.9, 91.2)
- added C22: 0.1uF, Capacitor_SMD:C_0603_1608Metric, F.Cu at (194.4, 90.8)
- added J1: Conn_01x05_Pin, Connector_PinHeader_2.54mm:PinHeader_1x05_P2.54mm_Vertical, F.Cu at (212.0, 52.5)
- added J10: Conn_01x01_Socket, Connector_Wire:SolderWirePad_1x01_SMD_2x4mm, F.Cu at (180.0, 116.5)
- added J2: Conn_01x01_Socket, Connector_Wire:SolderWirePad_1x01_SMD_3x6mm, F.Cu at (173.5, 27.5)
- added J3: Conn_01x01_Socket, Connector_Wire:SolderWirePad_1x01_SMD_3x6mm, F.Cu at (178.1, 27.5)
- added J4: Conn_01x01_Socket, Connector_Wire:SolderWirePad_1x01_SMD_3x6mm, F.Cu at (186.9, 117.0)
- added J5: Conn_01x01_Socket, Connector_Wire:SolderWirePad_1x01_SMD_3x6mm, F.Cu at (191.4, 117.0)
- added J6: Conn_01x01_Socket, Connector_Wire:SolderWirePad_1x01_SMD_3x6mm, F.Cu at (196.0, 117.0)
- added J7: Conn_01x01_Socket, Connector_Wire:SolderWirePad_1x01_SMD_2x4mm, F.Cu at (186.0, 27.5)
- added J8: Conn_01x01_Socket, Connector_Wire:SolderWirePad_1x01_SMD_2x4mm, F.Cu at (172.9, 116.5)
- added J9: Conn_01x01_Socket, Connector_Wire:SolderWirePad_1x01_SMD_2x4mm, F.Cu at (176.4, 116.5)
- added R6: 10k, Resistor_SMD:R_0603_1608Metric, F.Cu at (209.8, 56.2)
- added U3: 3.3V Regurator, Package_TO_SOT_SMD:SOT-89-3, F.Cu at (185.0, 38.5)
- C10, C11, C12, R4: moved to B.Cu
- Q2, Q3, Q6: moved to F.Cu
- moved C1 113.5 mm to (217.2, 69.8)
- moved C13 109.0 mm to (217.2, 73.3)
- moved C2 107.3 mm to (210.2, 76.8)
- moved C14 104.9 mm to (213.8, 62.8)
- moved C3 98.5 mm to (202.3, 73.8)
- moved C12 96.8 mm to (201.4, 87.5), turned to 90 degrees
- moved C15 93.6 mm to (202.5, 67.8)
- moved C6 87.5 mm to (191.8, 56.0)
- moved C4 87.2 mm to (192.0, 66.0)
- moved C11 86.9 mm to (189.9, 87.8), turned to 90 degrees
- moved C5 86.1 mm to (190.8, 69.0), turned to 180 degrees
- moved C8 83.8 mm to (187.3, 67.5), turned to 180 degrees
- moved C7 79.1 mm to (186.3, 65.5)
- moved R1 78.4 mm to (191.3, 52.0), turned to -90 degrees
- moved C10 78.1 mm to (179.4, 87.3), turned to 90 degrees
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Connections:
- C1 pad 1: GND -> SNA
- C13 pad 1: GND -> SNA
- C14 pad 1: GND -> SNA
- C15 pad 1: GND -> SNA
- C2 pad 1: GND -> SNA
- C3 pad 1: GND -> SNA
- Q1 pad 1: Net-(Q1-S) -> MOTOR_A
- Q2 pad 3: Net-(Q1-S) -> MOTOR_A
- Q3 pad 1: Net-(Q3-S) -> MOTOR_B
- Q4 pad 3: Net-(Q3-S) -> MOTOR_B
- Q5 pad 1: Net-(Q5-S) -> MOTOR_C
- Q6 pad 3: Net-(Q5-S) -> MOTOR_C
- U2 pad 14: GND -> SNA
- U2 pad 19: GND -> SNA
- U2 pad 21: SDO -> unconnected-(U2-PGD1/AD1AN5/CMP1C/ISRC0/IBIAS0/RP20/SDA1/RB3-Pad21)
- U2 pad 22: SDI -> unconnected-(U2-PGC1/AD2AN5/CMP2C/ISRC1/IBIAS1/RP21/SCL1/RB4-Pad22)
- U2 pad 23: SCLK -> unconnected-(U2-AD1ANN2/AD1AN8/RP23/RB6-Pad23)
- U2 pad 24: nCS -> unconnected-(U2-AD2ANN2/AD2AN8/RP24/IOMF0/RB7-Pad24)
- U2 pad 29: GND -> SNA
- U2 pad 35: GND -> SNA
- U2 pad 45: GND -> SNA
- U2 pad 6: GND -> SNA
Other:
- board outline removed

Commit message: update
Parts:
- added REF**: MountingHole_3.2mm_M3_ISO7380, MountingHole:MountingHole_3.2mm_M3_ISO7380, F.Cu at (167.0, 90.7)
- added REF**: MountingHole_3.2mm_M3_ISO7380, MountingHole:MountingHole_3.2mm_M3_ISO7380, F.Cu at (141.7, 80.6)
- C10, C11, C12: moved to F.Cu
- C17, C21, C22: moved to B.Cu
- moved C12 59.0 mm to (151.3, 56.4)
- moved C11 47.1 mm to (151.8, 60.1), turned to -90 degrees
- moved R5 45.7 mm to (157.2, 67.1)
- moved U1 44.9 mm to (145.2, 58.1)
- moved J4 44.6 mm to (151.1, 90.2)
- moved J6 44.6 mm to (160.2, 90.2)
- moved J5 44.6 mm to (155.7, 90.2)
- moved C4 43.8 mm to (148.3, 63.9)
- moved C5 43.8 mm to (147.1, 66.9)
- moved C6 43.8 mm to (148.0, 53.9)
- moved C7 43.8 mm to (142.6, 63.4)
- moved C8 43.8 mm to (143.5, 65.4)
- moved C9 43.8 mm to (139.5, 56.9)
- moved R1 43.8 mm to (147.5, 49.9)
- moved R2 43.8 mm to (145.0, 49.9)
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Other:
- board outline added: 40 x 50.7 mm

Commit message: dsaf
Parts:
- moved J2 45.0 mm to (133.1, 47.3)
- moved J7 34.2 mm to (157.7, 46.8)
- moved J3 22.2 mm to (167.8, 47.2)
- moved REF** 12.8 mm to (133.8, 90.7)
- moved R3 5.55 mm to (147.0, 64.8)
- moved R4 5.55 mm to (154.7, 65.0)
- moved R5 5.55 mm to (162.4, 65.0)
- moved C17 4.69 mm to (144.4, 75.9)
- moved C21 4.69 mm to (152.1, 76.0)
- moved C22 4.69 mm to (160.0, 75.9)
- moved J10 2.89 mm to (144.1, 91.3)
- moved J9 2.19 mm to (141.3, 91.3)
- moved J6 1.53 mm to (161.8, 90.3)
- moved J4 1.48 mm to (149.7, 90.3)
- moved J8 1.48 mm to (138.4, 91.3)
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Routing:
- added copper zone on F.Cu, net MOTOR_A

Commit message: upda
Parts:
- C17, C21, C22: moved to F.Cu
- U3: moved to B.Cu
- moved U3 57.0 mm to (129.9, 53.0), turned to 0 degrees
- moved C13 50.8 mm to (128.1, 70.2), turned to -45 degrees
- moved C1 46.3 mm to (134.2, 73.1)
- moved C2 44.4 mm to (127.2, 62.7), turned to -135 degrees
- moved C14 43.0 mm to (137.2, 73.1)
- moved U2 38.7 mm to (133.1, 65.9), turned to 45 degrees
- moved J2 34.8 mm to (167.8, 47.2)
- moved J7 29.6 mm to (128.1, 46.6)
- moved C3 26.9 mm to (137.1, 58.5), turned to 135 degrees
- moved J3 25.3 mm to (142.6, 47.2)
- moved C15 24.7 mm to (139.2, 60.6), turned to 135 degrees
- moved C5 13.6 mm to (158.8, 59.9), turned to -135 degrees
- moved C8 12.4 mm to (155.2, 61.4), turned to -135 degrees
- moved C4 11.5 mm to (157.5, 57.0), turned to 45 degrees
- moved J10 11.2 mm to (133.0, 90.8)
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Connections:
- U2 pad 10: SOB -> HB
- U2 pad 12: SOC -> HC
- U2 pad 13: HC -> unconnected-(U2-OA3IN+/AD2AN2/CMP3B/RP22/RB5-Pad13)
- U2 pad 16: HB -> SOA
- U2 pad 18: unconnected-(U2-OA2IN+/AD2AN4/CMP2B/RP19/RB2-Pad18) -> SOB
- U2 pad 22: unconnected-(U2-PGC1/AD2AN5/CMP2C/ISRC1/IBIAS1/RP21/SCL1/RB4-Pad22) -> SOC
- U2 pad 8: SOA -> HA
- U2 pad 9: HA -> unconnected-(U2-OA1IN-/AD1ANN1/AD2AN0/RP4/RA3-Pad9)
Routing:
- net SOB: track 0.00 -> 21.9 mm
- net SOA: track 0.00 -> 21.9 mm
- net SOC: track 0.00 -> 19.8 mm
- net INHA: track 0.00 -> 14.1 mm, vias 0 -> 2
- net INLA: track 0.00 -> 14.1 mm, vias 0 -> 2
- net INLB: track 0.00 -> 13.3 mm, vias 0 -> 2
- net INHB: track 0.00 -> 12.2 mm, vias 0 -> 2
- net INHC: track 0.00 -> 11.1 mm, vias 0 -> 2
- net INLC: track 0.00 -> 11.0 mm, vias 0 -> 2
- net HA: track 0.00 -> 5.65 mm
- net +3.3V: track 0.00 -> 5.10 mm, vias 0 -> 3
- net SNA: track 0.00 -> 4.71 mm, vias 0 -> 1
- net Net-(U1-DVDD): track 0.00 -> 3.33 mm
- net SPC: vias 0 -> 20
- net SPB: vias 0 -> 20
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- added copper zone on F.Cu, net MOTOR_B
- added copper zone on F.Cu, net MOTOR_C
- added copper zone on B.Cu, net SPA
- added copper zone on F.Cu, net SPA
- added copper zone on B.Cu, net SPB
- added copper zone on F.Cu, net SPB
- added copper zone on B.Cu, net SPC
- added copper zone on F.Cu, net SPC
Other:
- board size 40 x 50.7 mm -> 50 x 50 mm
- board text added: "A"
- board text added: "B"
- board text added: "C"

Commit message: up
Parts:
- removed C19: 10uF, Capacitor_SMD:C_Elec_5x5.4
- removed U3: 3.3V Regurator, Package_TO_SOT_SMD:SOT-89-3
- added C23: 1uF, Capacitor_SMD:C_0805_2012Metric, F.Cu at (127.5, 26.7)
- added C24: 1uF, Capacitor_SMD:C_0805_2012Metric, F.Cu at (127.5, 29.7)
- added J11: Conn_01x01_Socket, Connector_Wire:SolderWirePad_1x01_SMD_2x4mm, F.Cu at (142.1, 22.4)
- added J12: Conn_01x01_Socket, Connector_Wire:SolderWirePad_1x01_SMD_2x4mm, F.Cu at (145.7, 22.4)
- added J13: Conn_01x01_Socket, Connector_Wire:SolderWirePad_1x01_SMD_2x4mm, F.Cu at (149.2, 22.4)
- added J14: Conn_01x01_Socket, Connector_Wire:SolderWirePad_1x01_SMD_2x4mm, F.Cu at (152.8, 22.4)
- added R7: 10k, Resistor_SMD:R_0603_1608Metric, F.Cu at (127.3, 35.0)
- added U4: 3.3V Regurator, Package_TO_SOT_SMD:SOT-23-5, F.Cu at (119.1, 34.3)
- added U5: FIN1019MTCX, Package_SO:TSSOP-14_4.4x5mm_P0.65mm, F.Cu at (120.9, 28.6)
- C18: value 10uF -> 0.1uF; footprint Capacitor_SMD:C_Elec_5x5.4 -> Capacitor_SMD:C_0603_1608Metric
- moved C18 57.7 mm to (127.3, 32.5), turned to 0 degrees
Connections:
- C18 pad 1: VDC -> +3.3V
- U2 pad 25: unconnected-(U2-RP39/RC6-Pad25) -> LVDS_DE
- U2 pad 26: unconnected-(U2-RP40/RC7-Pad26) -> LVDS_DI
- U2 pad 27: unconnected-(U2-OSCO/CLKO/RP33/IOMF5/RC0-Pad27) -> LVDS_RE
- U2 pad 28: unconnected-(U2-OSCI/CLKI/RP34/IOMF6/RC1-Pad28) -> LVDS_RO

Commit message: dg
Parts:
- removed Q4, Q5, Q6: N-MOSFET, NTMFS5C468NLT1G:NTMFS5C468NLT1G
- C17, C21, C22: moved to B.Cu
- Q1, Q2, Q3: value N-MOSFET -> N-MOS Half-Bridge; footprint NTMFS5C468NLT1G:NTMFS5C468NLT1G -> CSD87588N:CSD87588N
- moved Q2 19.1 mm to (163.9, 80.9), turned to 0 degrees
- moved C17 18.7 mm to (159.1, 79.7)
- moved Q3 17.5 mm to (170.9, 80.9)
- moved C21 16.1 mm to (166.2, 79.6)
- moved Q1 13.6 mm to (156.9, 80.9)
- moved C22 12.9 mm to (173.2, 76.6)
- moved J4 12.0 mm to (156.7, 89.8)
- moved R3 10.7 mm to (153.3, 74.3)
- moved R4 8.66 mm to (160.4, 74.2)
- moved J5 7.09 mm to (161.5, 89.8)
- moved R5 6.99 mm to (167.4, 74.2)
- moved J6 2.23 mm to (166.3, 89.8)
Connections:
- Q1 pad 1: MOTOR_A -> GHA
- Q1 pad 2: GHA -> +BATT
- Q1 pad 3: +BATT -> SPA
- Q2 pad 1: SPA -> GHB
- Q2 pad 2: GLA -> +BATT
- Q2 pad 3: MOTOR_A -> SPB
- Q3 pad 1: MOTOR_B -> GHC
- Q3 pad 2: GHB -> +BATT
- Q3 pad 3: +BATT -> SPC
Routing:
- net SPC: vias 20 -> 0
- net SPB: vias 20 -> 0
- net SPA: vias 20 -> 0
- net MOTOR_C: vias 0 -> 12
- net MOTOR_B: vias 0 -> 12
- net MOTOR_A: vias 0 -> 12
- added copper zone on In1.Cu, net MOTOR_A
- added copper zone on In2.Cu, net MOTOR_A
- added copper zone on In3.Cu, net MOTOR_A
- added copper zone on In1.Cu, net MOTOR_B
- added copper zone on In2.Cu, net MOTOR_B
- added copper zone on In3.Cu, net MOTOR_B
- added copper zone on In1.Cu, net MOTOR_C
- added copper zone on In2.Cu, net MOTOR_C
- added copper zone on In3.Cu, net MOTOR_C
- removed copper zone on B.Cu, net SPA
- removed copper zone on F.Cu, net SPA
- removed copper zone on B.Cu, net SPB
- removed copper zone on F.Cu, net SPB
- removed copper zone on B.Cu, net SPC
- removed copper zone on F.Cu, net SPC
Other:
- copper layers 2 -> 8

Commit message: ap
Parts:
- R3, R4, R5: moved to F.Cu
- moved C2 43.7 mm to (170.7, 66.5), turned to 45 degrees
- moved C13 43.2 mm to (169.8, 59.0), turned to 135 degrees
- moved C1 34.1 mm to (163.8, 56.1), turned to 180 degrees
- moved U2 31.9 mm to (164.9, 63.4), turned to -135 degrees
- moved C14 29.1 mm to (160.8, 56.2), turned to 180 degrees
- moved C3 26.8 mm to (160.9, 70.8), turned to -45 degrees
- moved J8 26.4 mm to (165.0, 90.0)
- moved J10 26.4 mm to (159.3, 90.0)
- moved J9 26.4 mm to (162.2, 90.0)
- moved C17 24.5 mm to (135.2, 74.4)
- moved C21 24.1 mm to (142.4, 75.9)
- moved C22 23.4 mm to (149.8, 75.8)
- moved Q1 21.6 mm to (135.3, 80.9)
- moved J4 21.3 mm to (135.3, 89.8)
- moved Q2 21.2 mm to (142.7, 80.9)
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Routing:
- net SNA: track 4.71 -> 37.0 mm, vias 1 -> 0
- net MOTOR_A: track 0.00 -> 31.9 mm, vias 12 -> 57
- net GLA: track 0.00 -> 29.6 mm, vias 0 -> 2
- net GHA: track 0.00 -> 25.3 mm
- net SOB: track 21.9 -> 0.00 mm
- net SOA: track 21.9 -> 0.00 mm
- net SPA: track 0.00 -> 20.8 mm, vias 0 -> 20
- net SOC: track 19.8 -> 0.00 mm
- net SPC: track 0.00 -> 14.1 mm, vias 0 -> 20
- net INHA: track 14.1 -> 0.00 mm, vias 2 -> 0
- net INLA: track 14.1 -> 0.00 mm, vias 2 -> 0
- net SPB: track 0.00 -> 13.8 mm, vias 0 -> 20
- net INLB: track 13.3 -> 0.00 mm, vias 2 -> 0
- net INHB: track 12.2 -> 0.00 mm, vias 2 -> 0
- net INHC: track 11.1 -> 0.00 mm, vias 2 -> 0
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- added copper zone on F.Cu, net +BATT
- added copper zone on In1.Cu, net +BATT
- added copper zone on In2.Cu, net +BATT
- added copper zone on In3.Cu, net +BATT
- added copper zone on F.Cu, net SPA
- added copper zone on In1.Cu, net SPA
- added copper zone on In2.Cu, net SPA
- added copper zone on In3.Cu, net SPA
- added copper zone on F.Cu, net SPB
- added copper zone on In1.Cu, net SPB
- added copper zone on In2.Cu, net SPB
- added copper zone on In3.Cu, net SPB
- added copper zone on F.Cu, net SPC
- added copper zone on In1.Cu, net SPC
- added copper zone on In2.Cu, net SPC
- added copper zone on In3.Cu, net SPC

Commit message: af
Parts:
- added J15: Conn_01x01_Socket, Connector_Wire:SolderWirePad_1x01_SMD_2x4mm, F.Cu at (167.5, 90.6)
- added J16: Conn_01x01_Socket, Connector_Wire:SolderWirePad_1x01_SMD_2x4mm, F.Cu at (156.5, 90.6)
- moved J2 40.0 mm to (127.8, 47.4)
- moved R7 36.2 mm to (163.3, 38.3)
- moved U4 36.2 mm to (155.2, 37.6)
- moved C18 36.2 mm to (163.3, 35.8)
- moved C23 36.2 mm to (163.6, 30.0)
- moved C24 36.2 mm to (163.6, 33.0)
- moved U5 36.2 mm to (156.9, 31.9)
- moved J3 28.9 mm to (171.5, 47.2)
- moved J7 17.0 mm to (145.1, 48.0)
- moved C17 7.62 mm to (128.2, 77.4), turned to -90 degrees
- moved C22 6.09 mm to (155.5, 77.9), turned to -90 degrees
- moved R3 5.39 mm to (134.0, 77.9)
- moved Q1 5.00 mm to (130.3, 80.9)
- moved C21 4.61 mm to (138.2, 77.8), turned to -90 degrees
- moved C10 3.49 mm to (139.3, 66.3)
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Connections:
- U2 pad 10: HB -> unconnected-(U2-OA1IN+/AD1AN1/CMP1B/RP5/RA4-Pad10)
- U2 pad 12: HC -> unconnected-(U2-OA3IN-/AD1AN2/RP7/RA6-Pad12)
- U2 pad 2: unconnected-(U2-AD1AN6/RP8/IOMF1/RA7-Pad2) -> HA
- U2 pad 5: unconnected-(U2-AD1ANN3/AD1AN9/RP10/RA9-Pad5) -> HB
- U2 pad 8: HA -> HC
Routing:
- net SNA: track 37.0 -> 60.2 mm, vias 0 -> 147
- net GLB: track 0.00 -> 20.9 mm, vias 0 -> 2
- net MOTOR_B: track 0.00 -> 20.0 mm, vias 55 -> 81
- net MOTOR_C: track 0.00 -> 18.7 mm, vias 55 -> 81
- net GLC: track 0.00 -> 18.3 mm, vias 0 -> 2
- net GHC: track 0.00 -> 16.9 mm, vias 0 -> 2
- net GHB: track 0.00 -> 16.9 mm, vias 0 -> 2
- net SPC: track 14.1 -> 25.5 mm, vias 20 -> 40
- net MOTOR_A: track 31.9 -> 25.2 mm, vias 57 -> 81
- net HA: track 5.65 -> 0.00 mm
- net SPB: track 13.8 -> 17.8 mm, vias 20 -> 40
- net SPA: track 20.8 -> 21.7 mm, vias 20 -> 40
- net GHA: track 25.3 -> 25.2 mm, vias 0 -> 2
- net +BATT: vias 25 -> 158
- added copper zone on B.Cu, net +BATT
- added copper zone on In4.Cu, net +BATT
- added copper zone on In5.Cu, net +BATT
- added copper zone on In6.Cu, net +BATT
- added copper zone on B.Cu, net MOTOR_A
- added copper zone on In4.Cu, net MOTOR_A
- added copper zone on In5.Cu, net MOTOR_A
- added copper zone on In6.Cu, net MOTOR_A
- added copper zone on B.Cu, net MOTOR_B
- added copper zone on In4.Cu, net MOTOR_B
- added copper zone on In5.Cu, net MOTOR_B
- added copper zone on In6.Cu, net MOTOR_B
- added copper zone on B.Cu, net MOTOR_C
- added copper zone on In4.Cu, net MOTOR_C
- added copper zone on In5.Cu, net MOTOR_C
- added copper zone on In6.Cu, net MOTOR_C
- added copper zone on B.Cu, net SNA
- added copper zone on F.Cu, net SNA
- added copper zone on In1.Cu, net SNA
- added copper zone on In2.Cu, net SNA
- added copper zone on In3.Cu, net SNA
- added copper zone on In4.Cu, net SNA
- added copper zone on In5.Cu, net SNA
- added copper zone on In6.Cu, net SNA
- added copper zone on B.Cu, net SPA
- added copper zone on In4.Cu, net SPA
- added copper zone on In5.Cu, net SPA
- added copper zone on In6.Cu, net SPA
- added copper zone on B.Cu, net SPB
- added copper zone on In4.Cu, net SPB
- added copper zone on In5.Cu, net SPB
- added copper zone on In6.Cu, net SPB
- added copper zone on B.Cu, net SPC
- added copper zone on In4.Cu, net SPC
- added copper zone on In5.Cu, net SPC
- added copper zone on In6.Cu, net SPC
