File: BLDC_MOTOR_DRIVER_V0.kicad_pcb (KiCad board)
At the start: 8 copper layers, 50 x 50 mm, 55 parts, among them J1 Conn_01x05_Pin, J10 Conn_01x01_Socket, J11 Conn_01x01_Socket, J12 Conn_01x01_Socket, J13 Conn_01x01_Socket, J14 Conn_01x01_Socket, J15 Conn_01x01_Socket, J16 Conn_01x01_Socket, J2 Conn_01x01_Socket, J3 Conn_01x01_Socket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

Commit message: update
Parts:
- added REF**: MountingHole_3.2mm_M3_ISO7380, MountingHole:MountingHole_3.2mm_M3_ISO7380, F.Cu at (140.1, 47.4)
- moved J1 77.1 mm to (135.1, 57.8)
- moved R6 67.7 mm to (142.1, 55.0), turned to 90 degrees
- moved J11 32.5 mm to (163.6, 46.8)
- moved J12 32.5 mm to (167.1, 46.8)
- moved C23 29.8 mm to (143.1, 51.7), turned to 180 degrees
- moved U5 25.0 mm to (165.7, 55.3), turned to 90 degrees
- moved J13 24.9 mm to (155.0, 46.7)
- moved J14 24.9 mm to (158.5, 46.7)
- moved C24 21.8 mm to (148.5, 48.7), turned to 90 degrees
- moved C2 20.3 mm to (156.8, 53.1), turned to 180 degrees
- moved C13 18.8 mm to (152.6, 68.1), turned to 90 degrees
- moved R7 17.8 mm to (147.4, 46.2), turned to 180 degrees
- moved C18 16.1 mm to (161.2, 51.8), turned to -90 degrees
- moved C1 15.5 mm to (155.5, 70.5), turned to 0 degrees
- moved U4 14.9 mm to (145.4, 48.9), turned to 180 degrees
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Connections:
- U2 pad 16: SOA -> HA
- U2 pad 18: SOB -> HB
- U2 pad 2: HA -> SOA
- U2 pad 22: SOC -> HC
- U2 pad 25: LVDS_DE -> LVDS_RE
- U2 pad 26: LVDS_DI -> LVDS_RO
- U2 pad 27: LVDS_RE -> LVDS_DI
- U2 pad 28: LVDS_RO -> LVDS_DE
- U2 pad 5: HB -> SOB
- U2 pad 8: HC -> SOC
Routing:
- net +3.3V: track 0.00 -> 137.1 mm, vias 0 -> 16
- net SNA: track 60.2 -> 162.6 mm, vias 147 -> 256
- net VDC: track 0.00 -> 59.5 mm, vias 0 -> 3
- net +BATT: track 0.00 -> 49.0 mm, vias 158 -> 259
- net INHC: track 0.00 -> 37.0 mm, vias 0 -> 2
- net INLC: track 0.00 -> 33.5 mm, vias 0 -> 2
- net nFAULT: track 0.00 -> 31.5 mm, vias 0 -> 3
- net PGC: track 0.00 -> 29.5 mm, vias 0 -> 1
- net INHB: track 0.00 -> 25.5 mm, vias 0 -> 2
- net HA: track 0.00 -> 24.8 mm, vias 0 -> 2
- net HB: track 0.00 -> 24.7 mm, vias 0 -> 2
- net HC: track 0.00 -> 24.7 mm, vias 0 -> 2
- net MCLR: track 0.00 -> 24.6 mm, vias 0 -> 2
- net PGD: track 0.00 -> 24.1 mm, vias 0 -> 1
- net ENABLE: track 0.00 -> 23.3 mm, vias 0 -> 2
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
Commit message: fgn
Parts:
- removed C20: 10uF, Capacitor_SMD:C_Elec_5x5.4
- added C19: 22uF, Capacitor_SMD:CP_Elec_5x5.3, B.Cu at (132.2, 47.5)
- C16: value 10uF -> 22uF; footprint Capacitor_SMD:C_Elec_5x5.4 -> Capacitor_SMD:CP_Elec_5x5.3
- moved C16 81.8 mm to (114.2, 51.0)

Commit message: up
Parts:
- added R8: 10k, Resistor_SMD:R_0603_1608Metric, F.Cu at (152.4, 55.4)
- C16: moved to B.Cu
- moved C16 25.5 mm to (135.0, 65.8), turned to -90 degrees
- moved U4 3.50 mm to (144.7, 52.3)
- moved R6 3.20 mm to (139.8, 57.1)
- moved C23 2.41 mm to (141.6, 53.6), turned to 90 degrees
- moved REF** 2.39 mm to (142.5, 47.5)
- moved J1 2.35 mm to (137.1, 59.0)
- moved C8 1.28 mm to (138.2, 62.3)
- moved C24 0.70 mm to (147.8, 48.8)
- moved C4 0.50 mm to (135.1, 65.3)
- moved C5 0.50 mm to (135.1, 62.3)
- moved R7 0.25 mm to (147.2, 46.2)
Connections:
- U2 pad 10: unconnected-(U2-OA1IN+/AD1AN1/CMP1B/RP5/RA4-Pad10) -> MCU_NC
- U2 pad 11: unconnected-(U2-OA3OUT/AD1AN3/CMP3A/RP6/RA5-Pad11) -> MCU_NC
- U2 pad 12: unconnected-(U2-OA3IN-/AD1AN2/RP7/RA6-Pad12) -> MCU_NC
- U2 pad 13: unconnected-(U2-OA3IN+/AD2AN2/CMP3B/RP22/RB5-Pad13) -> MCU_NC
- U2 pad 17: unconnected-(U2-TMS/OA2IN-/AD1AN4/AD2ANN1/RP18/RB1-Pad17) -> MCU_NC
- U2 pad 21: unconnected-(U2-PGD1/AD1AN5/CMP1C/ISRC0/IBIAS0/RP20/SDA1/RB3-Pad21) -> MCU_NC
- U2 pad 23: unconnected-(U2-AD1ANN2/AD1AN8/RP23/RB6-Pad23) -> MCU_NC
- U2 pad 24: unconnected-(U2-AD2ANN2/AD2AN8/RP24/IOMF0/RB7-Pad24) -> MCU_NC
- U2 pad 4: unconnected-(U2-AD2AN9/ISRC3/IBIAS3/RP9/RA8-Pad4) -> MCU_NC
- U2 pad 47: unconnected-(U2-RP53/PCI22/RD4-Pad47) -> MCU_NC
- U2 pad 9: unconnected-(U2-OA1IN-/AD1ANN1/AD2AN0/RP4/RA3-Pad9) -> MCU_NC
Routing:
- net MCU_NC: track 0.00 -> 39.0 mm, vias 0 -> 6
- net VDC: track 59.5 -> 83.1 mm, vias 3 -> 19
- net Net-(U4-EN): track 1.76 -> 5.34 mm
- net PGC: track 29.5 -> 27.1 mm
- net PGD: track 24.1 -> 21.8 mm
- net MCLR: track 24.6 -> 22.4 mm
- net +3.3V: track 137.1 -> 135.1 mm
- net Net-(U1-VCP): track 4.27 -> 3.09 mm
- net +BATT: track 49.0 -> 49.3 mm, vias 259 -> 260
- net SNA: track 162.6 -> 162.8 mm, vias 256 -> 546
Other:
- board text added: "5V"
- board text added: "BATT+"
- board text added: "BATT-"
- board text added: "GND"
- board text added: "HA"
- board text added: "HB"
- board text added: "HC"
- board text added: "R+"
- board text added: "R-"
- board text added: "T+"
- board text added: "T-"

Commit message: v1.0.0
Parts:
- added R9: 100, Resistor_SMD:R_0402_1005Metric, B.Cu at (166.7, 55.8)
Routing:
- net LVDS_RI-: track 6.91 -> 10.4 mm, vias 0 -> 1
- net LVDS_RI+: track 7.39 -> 10.9 mm, vias 0 -> 1
- net SNA: vias 546 -> 547
