File: BLDC_MOTOR_DRIVER_ALPHA.kicad_pcb (KiCad board)
At the start: 8 copper layers, 50 x 50 mm, 58 parts, among them J1 Conn_01x05_Pin, J10 Conn_01x01_Socket, J11 Conn_01x01_Socket, J12 Conn_01x01_Socket, J13 Conn_01x01_Socket, J14 Conn_01x01_Socket, J15 Conn_01x01_Socket, J16 Conn_01x01_Socket, J2 Conn_01x01_Socket, J3 Conn_01x01_Socket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

Commit message: UPG
Parts:
- added JP1: Jumper_2_Small_Bridged, Resistor_SMD:R_0402_1005Metric, B.Cu at (127.9, 79.4)
- added JP2: Jumper_2_Small_Bridged, Resistor_SMD:R_0402_1005Metric, B.Cu at (127.2, 82.0)
- added JP3: Jumper_2_Small_Bridged, Resistor_SMD:R_0402_1005Metric, B.Cu at (138.9, 79.5)
- added JP4: Jumper_2_Small_Bridged, Resistor_SMD:R_0402_1005Metric, B.Cu at (138.3, 81.9)
- added JP5: Jumper_2_Small_Bridged, Resistor_SMD:R_0402_1005Metric, B.Cu at (149.2, 79.5)
- added JP6: Jumper_2_Small_Bridged, Resistor_SMD:R_0402_1005Metric, B.Cu at (148.6, 81.9)
Connections:
- Q1 pad 1: GHA -> Net-(JP1-B)
- Q1 pad 4: GLA -> Net-(JP2-B)
- Q2 pad 1: GHB -> Net-(JP3-B)
- Q2 pad 4: GLB -> Net-(JP4-B)
- Q3 pad 1: GHC -> Net-(JP5-B)
- Q3 pad 4: GLC -> Net-(JP6-B)
Routing:
- net GLB: track 20.9 -> 18.6 mm
- net Net-(JP2-B): track 0.00 -> 1.94 mm, vias 0 -> 1
- net GHC: track 16.9 -> 15.1 mm
- net GLA: track 29.4 -> 27.6 mm
- net GLC: track 18.3 -> 16.7 mm
- net Net-(JP1-B): track 0.00 -> 1.32 mm, vias 0 -> 1
- net Net-(JP6-B): track 0.00 -> 1.30 mm, vias 0 -> 1
- net Net-(JP4-B): track 0.00 -> 1.09 mm, vias 0 -> 1
- net Net-(JP5-B): track 0.00 -> 1.00 mm, vias 0 -> 1
- net MOTOR_C: track 18.7 -> 19.7 mm
- net Net-(JP3-B): track 0.00 -> 0.86 mm, vias 0 -> 1
- net SNA: vias 547 -> 551

Commit message: update
Parts:
- added G***: LOGO, global_footprints:icon_small_8.0x5.0, F.Cu at (171.8, 78.1)
Other:
- board text added: "BLDC"
