File: BLDC_MOTOR_DRIVER_ALPHA.kicad_sch (KiCad schematic)
At the start: 55 parts, among them J1 Conn_01x05_Pin, J10 Conn_01x01_Socket, J11 Conn_01x01_Socket, J12 Conn_01x01_Socket, J13 Conn_01x01_Socket, J14 Conn_01x01_Socket, J15 Conn_01x01_Socket, J16 Conn_01x01_Socket, J2 Conn_01x01_Socket, J3 Conn_01x01_Socket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

Commit message: UPG
Parts:
- added JP1, JP2, JP3, JP4, JP5, JP6: Jumper_2_Small_Bridged, Resistor_SMD:R_0402_1005Metric, symbol Jumper:Jumper_2_Small_Bridged
Connections:
- net GHA: now also JP1.1 (A); no longer Q1.1 (TG)
- net GHB: now also JP3.1 (A); no longer Q2.1 (TG)
- net GHC: now also JP5.1 (A); no longer Q3.1 (TG)
- net GLA: now also JP2.1 (A); no longer Q1.4 (BG)
- net GLB: now also JP4.1 (A); no longer Q2.4 (BG)
- net GLC: now also JP6.1 (A); no longer Q3.4 (BG)
- new net: JP2.2 (B), Q1.4 (BG)
- new net: JP5.2 (B), Q3.1 (TG)
- new net: JP4.2 (B), Q2.4 (BG)
- new net: JP3.2 (B), Q2.1 (TG)
- new net: JP6.2 (B), Q3.4 (BG)
- new net: JP1.2 (B), Q1.1 (TG)

Commit message: update
Parts:
- JP1, JP2, JP3, JP4, JP5, JP6: now left out of the parts list
Changed lines of the file:
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@@
 		(unit 1)
 		(exclude_from_sim no)
-		(in_bom yes)
+		(in_bom no)
 		(on_board yes)
 		(dnp no)
@@
 		(unit 1)
 		(exclude_from_sim no)
-		(in_bom yes)
+		(in_bom no)
 		(on_board yes)
 		(dnp no)
@@
 		(unit 1)
 		(exclude_from_sim no)
-		(in_bom yes)
+		(in_bom no)
 		(on_board yes)
 		(dnp no)
@@
 		(unit 1)
 		(exclude_from_sim no)
-		(in_bom yes)
+		(in_bom no)
 		(on_board yes)
 		(dnp no)
@@
 		(unit 1)
 		(exclude_from_sim no)
-		(in_bom yes)
+		(in_bom no)
 		(on_board yes)
 		(dnp no)
@@
 			)
 		)
-		(property "digikry" ""
-			(at 140.97 119.38 0)
-			(effects
-				(font
-					(size 1.27 1.27)
-				)
-				(hide yes)
-			)
-		)
 		(pin "2"
 		)
@@
 		(unit 1)
 		(exclude_from_sim no)
-		(in_bom yes)
+		(in_bom no)
 		(on_board yes)
 		(dnp no)
